Commit message: added motors and motor_test

File: test.urdf (robot description, URDF)
Before this commit: robot pepe, 36 links, 35 joints
Links:
- removed link 111
- removed link 16
- removed link 216
- removed link 221
- removed link 226
- removed link 231
- removed link 317
- removed link 319
- removed link 320
- removed link 322
- removed link 323
- removed link 325
- removed link 327
- removed link 328
- removed link 330
- removed link 332
- removed link 333
- removed link 335
- removed link 413
- removed link 42
- removed link 43
- removed link 48
- added link 144, mass 0.033049315320639795; collision cylinder length=0.3102879990410935 radius=0.184129683904798; visual cylinder length=0.3102879990410935 radius=0.184129683904798
- added link 22, mass 0.2343536963022129; collision cylinder length=0.15006793361516757 radius=0.7050452909954497; visual cylinder length=0.15006793361516757 radius=0.7050452909954497
- added link 223, mass 0.2343536963022129; collision cylinder length=0.15006793361516757 radius=0.7050452909954497; visual cylinder length=0.15006793361516757 radius=0.7050452909954497
- added link 245, mass 0.2343536963022129; collision cylinder length=0.15006793361516757 radius=0.7050452909954497; visual cylinder length=0.15006793361516757 radius=0.7050452909954497
- added link 266, mass 0.2343536963022129; collision cylinder length=0.15006793361516757 radius=0.7050452909954497; visual cylinder length=0.15006793361516757 radius=0.7050452909954497
- added link 313, mass 0.006208050542716708; collision cylinder length=0.29550920641413336 radius=0.08177436452571418; visual cylinder length=0.29550920641413336 radius=0.08177436452571418
- added link 33, mass 0.006208050542716708; collision cylinder length=0.29550920641413336 radius=0.08177436452571418; visual cylinder length=0.29550920641413336 radius=0.08177436452571418
- added link 339, mass 0.006208050542716708; collision cylinder length=0.29550920641413336 radius=0.08177436452571418; visual cylinder length=0.29550920641413336 radius=0.08177436452571418
- added link 346, mass 0.006208050542716708; collision cylinder length=0.29550920641413336 radius=0.08177436452571418; visual cylinder length=0.29550920641413336 radius=0.08177436452571418
- added link 351, mass 0.006208050542716708; collision cylinder length=0.29550920641413336 radius=0.08177436452571418; visual cylinder length=0.29550920641413336 radius=0.08177436452571418
- added link 356, mass 0.006208050542716708; collision cylinder length=0.29550920641413336 radius=0.08177436452571418; visual cylinder length=0.29550920641413336 radius=0.08177436452571418
- added link 361, mass 0.006208050542716708; collision cylinder length=0.29550920641413336 radius=0.08177436452571418; visual cylinder length=0.29550920641413336 radius=0.08177436452571418
- added link 367, mass 0.006208050542716708; collision cylinder length=0.29550920641413336 radius=0.08177436452571418; visual cylinder length=0.29550920641413336 radius=0.08177436452571418
- added link 372, mass 0.006208050542716708; collision cylinder length=0.29550920641413336 radius=0.08177436452571418; visual cylinder length=0.29550920641413336 radius=0.08177436452571418
- added link 377, mass 0.006208050542716708; collision cylinder length=0.29550920641413336 radius=0.08177436452571418; visual cylinder length=0.29550920641413336 radius=0.08177436452571418
- added link 38, mass 0.006208050542716708; collision cylinder length=0.29550920641413336 radius=0.08177436452571418; visual cylinder length=0.29550920641413336 radius=0.08177436452571418
- added link 382, mass 0.006208050542716708; collision cylinder length=0.29550920641413336 radius=0.08177436452571418; visual cylinder length=0.29550920641413336 radius=0.08177436452571418
- added link 411, mass 0.7345478185280645; collision cylinder length=0.6669404469852471 radius=0.5920952433820864; visual cylinder length=0.6669404469852471 radius=0.5920952433820864
- added link 416, mass 0.7345478185280645; collision cylinder length=0.6669404469852471 radius=0.5920952433820864; visual cylinder length=0.6669404469852471 radius=0.5920952433820864
- added link 417, mass 0.7345478185280645; collision cylinder length=0.6669404469852471 radius=0.5920952433820864; visual cylinder length=0.6669404469852471 radius=0.5920952433820864
- added link 419, mass 0.7345478185280645; collision cylinder length=0.6669404469852471 radius=0.5920952433820864; visual cylinder length=0.6669404469852471 radius=0.5920952433820864
- added link 420, mass 0.7345478185280645; collision cylinder length=0.6669404469852471 radius=0.5920952433820864; visual cylinder length=0.6669404469852471 radius=0.5920952433820864
- added link 421, mass 0.7345478185280645; collision cylinder length=0.6669404469852471 radius=0.5920952433820864; visual cylinder length=0.6669404469852471 radius=0.5920952433820864
- added link 422, mass 0.7345478185280645; collision cylinder length=0.6669404469852471 radius=0.5920952433820864; visual cylinder length=0.6669404469852471 radius=0.5920952433820864
- added link 425, mass 0.7345478185280645; collision cylinder length=0.6669404469852471 radius=0.5920952433820864; visual cylinder length=0.6669404469852471 radius=0.5920952433820864
- added link 426, mass 0.7345478185280645; collision cylinder length=0.6669404469852471 radius=0.5920952433820864; visual cylinder length=0.6669404469852471 radius=0.5920952433820864
- added link 427, mass 0.7345478185280645; collision cylinder length=0.6669404469852471 radius=0.5920952433820864; visual cylinder length=0.6669404469852471 radius=0.5920952433820864
- added link 428, mass 0.7345478185280645; collision cylinder length=0.6669404469852471 radius=0.5920952433820864; visual cylinder length=0.6669404469852471 radius=0.5920952433820864
- added link 430, mass 0.7345478185280645; collision cylinder length=0.6669404469852471 radius=0.5920952433820864; visual cylinder length=0.6669404469852471 radius=0.5920952433820864
- added link 431, mass 0.7345478185280645; collision cylinder length=0.6669404469852471 radius=0.5920952433820864; visual cylinder length=0.6669404469852471 radius=0.5920952433820864
- added link 432, mass 0.7345478185280645; collision cylinder length=0.6669404469852471 radius=0.5920952433820864; visual cylinder length=0.6669404469852471 radius=0.5920952433820864
- added link 433, mass 0.7345478185280645; collision cylinder length=0.6669404469852471 radius=0.5920952433820864; visual cylinder length=0.6669404469852471 radius=0.5920952433820864
- added link 435, mass 0.7345478185280645; collision cylinder length=0.6669404469852471 radius=0.5920952433820864; visual cylinder length=0.6669404469852471 radius=0.5920952433820864
- added link 436, mass 0.7345478185280645; collision cylinder length=0.6669404469852471 radius=0.5920952433820864; visual cylinder length=0.6669404469852471 radius=0.5920952433820864
- added link 437, mass 0.7345478185280645; collision cylinder length=0.6669404469852471 radius=0.5920952433820864; visual cylinder length=0.6669404469852471 radius=0.5920952433820864
- added link 438, mass 0.7345478185280645; collision cylinder length=0.6669404469852471 radius=0.5920952433820864; visual cylinder length=0.6669404469852471 radius=0.5920952433820864
- added link 440, mass 0.7345478185280645; collision cylinder length=0.6669404469852471 radius=0.5920952433820864; visual cylinder length=0.6669404469852471 radius=0.5920952433820864
- added link 441, mass 0.7345478185280645; collision cylinder length=0.6669404469852471 radius=0.5920952433820864; visual cylinder length=0.6669404469852471 radius=0.5920952433820864
- added link 442, mass 0.7345478185280645; collision cylinder length=0.6669404469852471 radius=0.5920952433820864; visual cylinder length=0.6669404469852471 radius=0.5920952433820864
- added link 443, mass 0.7345478185280645; collision cylinder length=0.6669404469852471 radius=0.5920952433820864; visual cylinder length=0.6669404469852471 radius=0.5920952433820864
- added link 447, mass 0.7345478185280645; collision cylinder length=0.6669404469852471 radius=0.5920952433820864; visual cylinder length=0.6669404469852471 radius=0.5920952433820864
- added link 448, mass 0.7345478185280645; collision cylinder length=0.6669404469852471 radius=0.5920952433820864; visual cylinder length=0.6669404469852471 radius=0.5920952433820864
- added link 449, mass 0.7345478185280645; collision cylinder length=0.6669404469852471 radius=0.5920952433820864; visual cylinder length=0.6669404469852471 radius=0.5920952433820864
- added link 450, mass 0.7345478185280645; collision cylinder length=0.6669404469852471 radius=0.5920952433820864; visual cylinder length=0.6669404469852471 radius=0.5920952433820864
- added link 452, mass 0.7345478185280645; collision cylinder length=0.6669404469852471 radius=0.5920952433820864; visual cylinder length=0.6669404469852471 radius=0.5920952433820864
- added link 453, mass 0.7345478185280645; collision cylinder length=0.6669404469852471 radius=0.5920952433820864; visual cylinder length=0.6669404469852471 radius=0.5920952433820864
- added link 454, mass 0.7345478185280645; collision cylinder length=0.6669404469852471 radius=0.5920952433820864; visual cylinder length=0.6669404469852471 radius=0.5920952433820864
- added link 455, mass 0.7345478185280645; collision cylinder length=0.6669404469852471 radius=0.5920952433820864; visual cylinder length=0.6669404469852471 radius=0.5920952433820864
- added link 457, mass 0.7345478185280645; collision cylinder length=0.6669404469852471 radius=0.5920952433820864; visual cylinder length=0.6669404469852471 radius=0.5920952433820864
- added link 458, mass 0.7345478185280645; collision cylinder length=0.6669404469852471 radius=0.5920952433820864; visual cylinder length=0.6669404469852471 radius=0.5920952433820864
- added link 459, mass 0.7345478185280645; collision cylinder length=0.6669404469852471 radius=0.5920952433820864; visual cylinder length=0.6669404469852471 radius=0.5920952433820864
- added link 46, mass 0.7345478185280645; collision cylinder length=0.6669404469852471 radius=0.5920952433820864; visual cylinder length=0.6669404469852471 radius=0.5920952433820864
- added link 460, mass 0.7345478185280645; collision cylinder length=0.6669404469852471 radius=0.5920952433820864; visual cylinder length=0.6669404469852471 radius=0.5920952433820864
- added link 462, mass 0.7345478185280645; collision cylinder length=0.6669404469852471 radius=0.5920952433820864; visual cylinder length=0.6669404469852471 radius=0.5920952433820864
- added link 463, mass 0.7345478185280645; collision cylinder length=0.6669404469852471 radius=0.5920952433820864; visual cylinder length=0.6669404469852471 radius=0.5920952433820864
- added link 464, mass 0.7345478185280645; collision cylinder length=0.6669404469852471 radius=0.5920952433820864; visual cylinder length=0.6669404469852471 radius=0.5920952433820864
- added link 465, mass 0.7345478185280645; collision cylinder length=0.6669404469852471 radius=0.5920952433820864; visual cylinder length=0.6669404469852471 radius=0.5920952433820864
- added link 468, mass 0.7345478185280645; collision cylinder length=0.6669404469852471 radius=0.5920952433820864; visual cylinder length=0.6669404469852471 radius=0.5920952433820864
- added link 469, mass 0.7345478185280645; collision cylinder length=0.6669404469852471 radius=0.5920952433820864; visual cylinder length=0.6669404469852471 radius=0.5920952433820864
- added link 470, mass 0.7345478185280645; collision cylinder length=0.6669404469852471 radius=0.5920952433820864; visual cylinder length=0.6669404469852471 radius=0.5920952433820864
- added link 471, mass 0.7345478185280645; collision cylinder length=0.6669404469852471 radius=0.5920952433820864; visual cylinder length=0.6669404469852471 radius=0.5920952433820864
- added link 473, mass 0.7345478185280645; collision cylinder length=0.6669404469852471 radius=0.5920952433820864; visual cylinder length=0.6669404469852471 radius=0.5920952433820864
- added link 474, mass 0.7345478185280645; collision cylinder length=0.6669404469852471 radius=0.5920952433820864; visual cylinder length=0.6669404469852471 radius=0.5920952433820864
- added link 475, mass 0.7345478185280645; collision cylinder length=0.6669404469852471 radius=0.5920952433820864; visual cylinder length=0.6669404469852471 radius=0.5920952433820864
- added link 476, mass 0.7345478185280645; collision cylinder length=0.6669404469852471 radius=0.5920952433820864; visual cylinder length=0.6669404469852471 radius=0.5920952433820864
- added link 478, mass 0.7345478185280645; collision cylinder length=0.6669404469852471 radius=0.5920952433820864; visual cylinder length=0.6669404469852471 radius=0.5920952433820864
- added link 479, mass 0.7345478185280645; collision cylinder length=0.6669404469852471 radius=0.5920952433820864; visual cylinder length=0.6669404469852471 radius=0.5920952433820864
- added link 480, mass 0.7345478185280645; collision cylinder length=0.6669404469852471 radius=0.5920952433820864; visual cylinder length=0.6669404469852471 radius=0.5920952433820864
- added link 481, mass 0.7345478185280645; collision cylinder length=0.6669404469852471 radius=0.5920952433820864; visual cylinder length=0.6669404469852471 radius=0.5920952433820864
- added link 483, mass 0.7345478185280645; collision cylinder length=0.6669404469852471 radius=0.5920952433820864; visual cylinder length=0.6669404469852471 radius=0.5920952433820864
- added link 484, mass 0.7345478185280645; collision cylinder length=0.6669404469852471 radius=0.5920952433820864; visual cylinder length=0.6669404469852471 radius=0.5920952433820864
- added link 485, mass 0.7345478185280645; collision cylinder length=0.6669404469852471 radius=0.5920952433820864; visual cylinder length=0.6669404469852471 radius=0.5920952433820864
- added link 486, mass 0.7345478185280645; collision cylinder length=0.6669404469852471 radius=0.5920952433820864; visual cylinder length=0.6669404469852471 radius=0.5920952433820864
- link 0: mass 0.30599540799876335 -> 0.0005252686028896167; geometry collision cylinder length=0.30747636043019333 radius=0.023318999813060626; visual cylinder length=0.30747636043019333 radius=0.023318999813060626
- link 11: mass 0.020145828931550726 -> 0.033049315320639795; geometry collision cylinder length=0.3102879990410935 radius=0.184129683904798; visual cylinder length=0.3102879990410935 radius=0.184129683904798
- link 318: mass 2.1035649095397932 -> 0.006208050542716708; geometry collision cylinder length=0.29550920641413336 radius=0.08177436452571418; visual cylinder length=0.29550920641413336 radius=0.08177436452571418
- link 324: mass 2.1035649095397932 -> 0.006208050542716708; geometry collision cylinder length=0.29550920641413336 radius=0.08177436452571418; visual cylinder length=0.29550920641413336 radius=0.08177436452571418
- link 329: mass 2.1035649095397932 -> 0.006208050542716708; geometry collision cylinder length=0.29550920641413336 radius=0.08177436452571418; visual cylinder length=0.29550920641413336 radius=0.08177436452571418
- link 334: mass 2.1035649095397932 -> 0.006208050542716708; geometry collision cylinder length=0.29550920641413336 radius=0.08177436452571418; visual cylinder length=0.29550920641413336 radius=0.08177436452571418
- link 410: mass 0.14757926132102542 -> 0.7345478185280645; geometry collision cylinder length=0.6669404469852471 radius=0.5920952433820864; visual cylinder length=0.6669404469852471 radius=0.5920952433820864
- link 412: mass 0.14757926132102542 -> 0.7345478185280645; geometry collision cylinder length=0.6669404469852471 radius=0.5920952433820864; visual cylinder length=0.6669404469852471 radius=0.5920952433820864
- link 414: mass 0.14757926132102542 -> 0.7345478185280645; geometry collision cylinder length=0.6669404469852471 radius=0.5920952433820864; visual cylinder length=0.6669404469852471 radius=0.5920952433820864
- link 415: mass 0.14757926132102542 -> 0.7345478185280645; geometry collision cylinder length=0.6669404469852471 radius=0.5920952433820864; visual cylinder length=0.6669404469852471 radius=0.5920952433820864
- link 44: mass 0.14757926132102542 -> 0.7345478185280645; geometry collision cylinder length=0.6669404469852471 radius=0.5920952433820864; visual cylinder length=0.6669404469852471 radius=0.5920952433820864
- link 45: mass 0.14757926132102542 -> 0.7345478185280645; geometry collision cylinder length=0.6669404469852471 radius=0.5920952433820864; visual cylinder length=0.6669404469852471 radius=0.5920952433820864
- link 47: mass 0.14757926132102542 -> 0.7345478185280645; geometry collision cylinder length=0.6669404469852471 radius=0.5920952433820864; visual cylinder length=0.6669404469852471 radius=0.5920952433820864
- link 49: mass 0.14757926132102542 -> 0.7345478185280645; geometry collision cylinder length=0.6669404469852471 radius=0.5920952433820864; visual cylinder length=0.6669404469852471 radius=0.5920952433820864
Joints:
- removed joint 111_to_0
- removed joint 16_to_0
- removed joint 216_to_0
- removed joint 221_to_0
- removed joint 226_to_0
- removed joint 231_to_0
- removed joint 317_to_216
- removed joint 318_to_216
- removed joint 319_to_216
- removed joint 320_to_216
- removed joint 322_to_221
- removed joint 323_to_221
- removed joint 324_to_221
- removed joint 325_to_221
- removed joint 327_to_226
- removed joint 328_to_226
- removed joint 329_to_226
- removed joint 330_to_226
- removed joint 332_to_231
- removed joint 333_to_231
- removed joint 334_to_231
- removed joint 335_to_231
- removed joint 410_to_16
- removed joint 412_to_111
- removed joint 413_to_111
- removed joint 414_to_111
- removed joint 415_to_111
- removed joint 42_to_11
- removed joint 43_to_11
- removed joint 44_to_11
- removed joint 45_to_11
- removed joint 47_to_16
- removed joint 48_to_16
- removed joint 49_to_16
- added joint 144_to_0: type revolute, parent 0, child 144, origin xyz=0.15038454251742672 0.9250536779485011 0.2625608772024355 rpy=5.036943397516115 6.158822008435018 5.754327538697678, axis 0 0 1, limit lower=3.1415 upper=-3.1415 effort=1 velocity=1
- added joint 223_to_11: type revolute, parent 11, child 223, origin xyz=0.06841846425951548 0.9729246395836781 0.5945876398141128 rpy=17.479377941547902 4.5103860222098895 0.24855167088342786, axis 0 1 0, limit lower=3.1415 upper=-3.1415 effort=1 velocity=1
- added joint 22_to_11: type revolute, parent 11, child 22, origin xyz=0.06841846425951548 0.9729246395836781 0.5945876398141128 rpy=11.6529186276986 4.5103860222098895 0.24855167088342786, axis 0 1 0, limit lower=3.1415 upper=-3.1415 effort=1 velocity=1
- added joint 245_to_144: type revolute, parent 144, child 245, origin xyz=0.06841846425951548 0.9729246395836781 0.5945876398141128 rpy=11.6529186276986 4.5103860222098895 0.24855167088342786, axis 0 1 0, limit lower=3.1415 upper=-3.1415 effort=1 velocity=1
- added joint 266_to_144: type revolute, parent 144, child 266, origin xyz=0.06841846425951548 0.9729246395836781 0.5945876398141128 rpy=17.479377941547902 4.5103860222098895 0.24855167088342786, axis 0 1 0, limit lower=3.1415 upper=-3.1415 effort=1 velocity=1
- added joint 313_to_22: type revolute, parent 22, child 313, origin xyz=0.4880510962654848 0.962889575441964 0.3859426861683787 rpy=3.949138026192128 2.36130074223153 4.3265520768295085, axis 0 1 0, limit lower=3.1415 upper=-3.1415 effort=1 velocity=1
- added joint 318_to_22: type revolute, parent 22, child 318, origin xyz=0.4880510962654848 0.962889575441964 0.3859426861683787 rpy=4.93642253274016 2.36130074223153 4.3265520768295085, axis 0 1 0, limit lower=3.1415 upper=-3.1415 effort=1 velocity=1
- added joint 324_to_223: type revolute, parent 223, child 324, origin xyz=0.4880510962654848 0.962889575441964 0.3859426861683787 rpy=1.974569013096064 2.36130074223153 4.3265520768295085, axis 0 1 0, limit lower=3.1415 upper=-3.1415 effort=1 velocity=1
- added joint 329_to_223: type revolute, parent 223, child 329, origin xyz=0.4880510962654848 0.962889575441964 0.3859426861683787 rpy=2.9618535196440963 2.36130074223153 4.3265520768295085, axis 0 1 0, limit lower=3.1415 upper=-3.1415 effort=1 velocity=1
- added joint 334_to_223: type revolute, parent 223, child 334, origin xyz=0.4880510962654848 0.962889575441964 0.3859426861683787 rpy=3.949138026192128 2.36130074223153 4.3265520768295085, axis 0 1 0, limit lower=3.1415 upper=-3.1415 effort=1 velocity=1
- added joint 339_to_223: type revolute, parent 223, child 339, origin xyz=0.4880510962654848 0.962889575441964 0.3859426861683787 rpy=4.93642253274016 2.36130074223153 4.3265520768295085, axis 0 1 0, limit lower=3.1415 upper=-3.1415 effort=1 velocity=1
- added joint 33_to_22: type revolute, parent 22, child 33, origin xyz=0.4880510962654848 0.962889575441964 0.3859426861683787 rpy=1.974569013096064 2.36130074223153 4.3265520768295085, axis 0 1 0, limit lower=3.1415 upper=-3.1415 effort=1 velocity=1
- added joint 346_to_245: type revolute, parent 245, child 346, origin xyz=0.4880510962654848 0.962889575441964 0.3859426861683787 rpy=1.974569013096064 2.36130074223153 4.3265520768295085, axis 0 1 0, limit lower=3.1415 upper=-3.1415 effort=1 velocity=1
- added joint 351_to_245: type revolute, parent 245, child 351, origin xyz=0.4880510962654848 0.962889575441964 0.3859426861683787 rpy=2.9618535196440963 2.36130074223153 4.3265520768295085, axis 0 1 0, limit lower=3.1415 upper=-3.1415 effort=1 velocity=1
- added joint 356_to_245: type revolute, parent 245, child 356, origin xyz=0.4880510962654848 0.962889575441964 0.3859426861683787 rpy=3.949138026192128 2.36130074223153 4.3265520768295085, axis 0 1 0, limit lower=3.1415 upper=-3.1415 effort=1 velocity=1
- added joint 361_to_245: type revolute, parent 245, child 361, origin xyz=0.4880510962654848 0.962889575441964 0.3859426861683787 rpy=4.93642253274016 2.36130074223153 4.3265520768295085, axis 0 1 0, limit lower=3.1415 upper=-3.1415 effort=1 velocity=1
- added joint 367_to_266: type revolute, parent 266, child 367, origin xyz=0.4880510962654848 0.962889575441964 0.3859426861683787 rpy=1.974569013096064 2.36130074223153 4.3265520768295085, axis 0 1 0, limit lower=3.1415 upper=-3.1415 effort=1 velocity=1
- added joint 372_to_266: type revolute, parent 266, child 372, origin xyz=0.4880510962654848 0.962889575441964 0.3859426861683787 rpy=2.9618535196440963 2.36130074223153 4.3265520768295085, axis 0 1 0, limit lower=3.1415 upper=-3.1415 effort=1 velocity=1
- added joint 377_to_266: type revolute, parent 266, child 377, origin xyz=0.4880510962654848 0.962889575441964 0.3859426861683787 rpy=3.949138026192128 2.36130074223153 4.3265520768295085, axis 0 1 0, limit lower=3.1415 upper=-3.1415 effort=1 velocity=1
- added joint 382_to_266: type revolute, parent 266, child 382, origin xyz=0.4880510962654848 0.962889575441964 0.3859426861683787 rpy=4.93642253274016 2.36130074223153 4.3265520768295085, axis 0 1 0, limit lower=3.1415 upper=-3.1415 effort=1 velocity=1
- added joint 38_to_22: type revolute, parent 22, child 38, origin xyz=0.4880510962654848 0.962889575441964 0.3859426861683787 rpy=2.9618535196440963 2.36130074223153 4.3265520768295085, axis 0 1 0, limit lower=3.1415 upper=-3.1415 effort=1 velocity=1
- added joint 410_to_38: type revolute, parent 38, child 410, origin xyz=0.5607100632388653 0.5633427228192782 0.10525246131887211 rpy=14.300179234301686 6.085246563263388 4.797191989166931, axis 0 1 0, limit lower=3.1415 upper=-3.1415 effort=1 velocity=1
- added joint 411_to_38: type revolute, parent 38, child 411, origin xyz=0.5607100632388653 0.5633427228192782 0.10525246131887211 rpy=19.06690564573558 6.085246563263388 4.797191989166931, axis 0 1 0, limit lower=3.1415 upper=-3.1415 effort=1 velocity=1
- added joint 412_to_38: type revolute, parent 38, child 412, origin xyz=0.5607100632388653 0.5633427228192782 0.10525246131887211 rpy=23.833632057169474 6.085246563263388 4.797191989166931, axis 0 1 0, limit lower=3.1415 upper=-3.1415 effort=1 velocity=1
- added joint 414_to_313: type revolute, parent 313, child 414, origin xyz=0.5607100632388653 0.5633427228192782 0.10525246131887211 rpy=9.53345282286779 6.085246563263388 4.797191989166931, axis 0 1 0, limit lower=3.1415 upper=-3.1415 effort=1 velocity=1
- added joint 415_to_313: type revolute, parent 313, child 415, origin xyz=0.5607100632388653 0.5633427228192782 0.10525246131887211 rpy=14.300179234301686 6.085246563263388 4.797191989166931, axis 0 1 0, limit lower=3.1415 upper=-3.1415 effort=1 velocity=1
- added joint 416_to_313: type revolute, parent 313, child 416, origin xyz=0.5607100632388653 0.5633427228192782 0.10525246131887211 rpy=19.06690564573558 6.085246563263388 4.797191989166931, axis 0 1 0, limit lower=3.1415 upper=-3.1415 effort=1 velocity=1
- added joint 417_to_313: type revolute, parent 313, child 417, origin xyz=0.5607100632388653 0.5633427228192782 0.10525246131887211 rpy=23.833632057169474 6.085246563263388 4.797191989166931, axis 0 1 0, limit lower=3.1415 upper=-3.1415 effort=1 velocity=1
- added joint 419_to_318: type revolute, parent 318, child 419, origin xyz=0.5607100632388653 0.5633427228192782 0.10525246131887211 rpy=9.53345282286779 6.085246563263388 4.797191989166931, axis 0 1 0, limit lower=3.1415 upper=-3.1415 effort=1 velocity=1
- added joint 420_to_318: type revolute, parent 318, child 420, origin xyz=0.5607100632388653 0.5633427228192782 0.10525246131887211 rpy=14.300179234301686 6.085246563263388 4.797191989166931, axis 0 1 0, limit lower=3.1415 upper=-3.1415 effort=1 velocity=1
- added joint 421_to_318: type revolute, parent 318, child 421, origin xyz=0.5607100632388653 0.5633427228192782 0.10525246131887211 rpy=19.06690564573558 6.085246563263388 4.797191989166931, axis 0 1 0, limit lower=3.1415 upper=-3.1415 effort=1 velocity=1
- added joint 422_to_318: type revolute, parent 318, child 422, origin xyz=0.5607100632388653 0.5633427228192782 0.10525246131887211 rpy=23.833632057169474 6.085246563263388 4.797191989166931, axis 0 1 0, limit lower=3.1415 upper=-3.1415 effort=1 velocity=1
- added joint 425_to_324: type revolute, parent 324, child 425, origin xyz=0.5607100632388653 0.5633427228192782 0.10525246131887211 rpy=9.53345282286779 6.085246563263388 4.797191989166931, axis 0 1 0, limit lower=3.1415 upper=-3.1415 effort=1 velocity=1
- added joint 426_to_324: type revolute, parent 324, child 426, origin xyz=0.5607100632388653 0.5633427228192782 0.10525246131887211 rpy=14.300179234301686 6.085246563263388 4.797191989166931, axis 0 1 0, limit lower=3.1415 upper=-3.1415 effort=1 velocity=1
- added joint 427_to_324: type revolute, parent 324, child 427, origin xyz=0.5607100632388653 0.5633427228192782 0.10525246131887211 rpy=19.06690564573558 6.085246563263388 4.797191989166931, axis 0 1 0, limit lower=3.1415 upper=-3.1415 effort=1 velocity=1
- added joint 428_to_324: type revolute, parent 324, child 428, origin xyz=0.5607100632388653 0.5633427228192782 0.10525246131887211 rpy=23.833632057169474 6.085246563263388 4.797191989166931, axis 0 1 0, limit lower=3.1415 upper=-3.1415 effort=1 velocity=1
- added joint 430_to_329: type revolute, parent 329, child 430, origin xyz=0.5607100632388653 0.5633427228192782 0.10525246131887211 rpy=9.53345282286779 6.085246563263388 4.797191989166931, axis 0 1 0, limit lower=3.1415 upper=-3.1415 effort=1 velocity=1
- added joint 431_to_329: type revolute, parent 329, child 431, origin xyz=0.5607100632388653 0.5633427228192782 0.10525246131887211 rpy=14.300179234301686 6.085246563263388 4.797191989166931, axis 0 1 0, limit lower=3.1415 upper=-3.1415 effort=1 velocity=1
- added joint 432_to_329: type revolute, parent 329, child 432, origin xyz=0.5607100632388653 0.5633427228192782 0.10525246131887211 rpy=19.06690564573558 6.085246563263388 4.797191989166931, axis 0 1 0, limit lower=3.1415 upper=-3.1415 effort=1 velocity=1
- added joint 433_to_329: type revolute, parent 329, child 433, origin xyz=0.5607100632388653 0.5633427228192782 0.10525246131887211 rpy=23.833632057169474 6.085246563263388 4.797191989166931, axis 0 1 0, limit lower=3.1415 upper=-3.1415 effort=1 velocity=1
- added joint 435_to_334: type revolute, parent 334, child 435, origin xyz=0.5607100632388653 0.5633427228192782 0.10525246131887211 rpy=9.53345282286779 6.085246563263388 4.797191989166931, axis 0 1 0, limit lower=3.1415 upper=-3.1415 effort=1 velocity=1
- added joint 436_to_334: type revolute, parent 334, child 436, origin xyz=0.5607100632388653 0.5633427228192782 0.10525246131887211 rpy=14.300179234301686 6.085246563263388 4.797191989166931, axis 0 1 0, limit lower=3.1415 upper=-3.1415 effort=1 velocity=1
- added joint 437_to_334: type revolute, parent 334, child 437, origin xyz=0.5607100632388653 0.5633427228192782 0.10525246131887211 rpy=19.06690564573558 6.085246563263388 4.797191989166931, axis 0 1 0, limit lower=3.1415 upper=-3.1415 effort=1 velocity=1
- added joint 438_to_334: type revolute, parent 334, child 438, origin xyz=0.5607100632388653 0.5633427228192782 0.10525246131887211 rpy=23.833632057169474 6.085246563263388 4.797191989166931, axis 0 1 0, limit lower=3.1415 upper=-3.1415 effort=1 velocity=1
- added joint 440_to_339: type revolute, parent 339, child 440, origin xyz=0.5607100632388653 0.5633427228192782 0.10525246131887211 rpy=9.53345282286779 6.085246563263388 4.797191989166931, axis 0 1 0, limit lower=3.1415 upper=-3.1415 effort=1 velocity=1
- added joint 441_to_339: type revolute, parent 339, child 441, origin xyz=0.5607100632388653 0.5633427228192782 0.10525246131887211 rpy=14.300179234301686 6.085246563263388 4.797191989166931, axis 0 1 0, limit lower=3.1415 upper=-3.1415 effort=1 velocity=1
- added joint 442_to_339: type revolute, parent 339, child 442, origin xyz=0.5607100632388653 0.5633427228192782 0.10525246131887211 rpy=19.06690564573558 6.085246563263388 4.797191989166931, axis 0 1 0, limit lower=3.1415 upper=-3.1415 effort=1 velocity=1
- added joint 443_to_339: type revolute, parent 339, child 443, origin xyz=0.5607100632388653 0.5633427228192782 0.10525246131887211 rpy=23.833632057169474 6.085246563263388 4.797191989166931, axis 0 1 0, limit lower=3.1415 upper=-3.1415 effort=1 velocity=1
- added joint 447_to_346: type revolute, parent 346, child 447, origin xyz=0.5607100632388653 0.5633427228192782 0.10525246131887211 rpy=9.53345282286779 6.085246563263388 4.797191989166931, axis 0 1 0, limit lower=3.1415 upper=-3.1415 effort=1 velocity=1
- added joint 448_to_346: type revolute, parent 346, child 448, origin xyz=0.5607100632388653 0.5633427228192782 0.10525246131887211 rpy=14.300179234301686 6.085246563263388 4.797191989166931, axis 0 1 0, limit lower=3.1415 upper=-3.1415 effort=1 velocity=1
- added joint 449_to_346: type revolute, parent 346, child 449, origin xyz=0.5607100632388653 0.5633427228192782 0.10525246131887211 rpy=19.06690564573558 6.085246563263388 4.797191989166931, axis 0 1 0, limit lower=3.1415 upper=-3.1415 effort=1 velocity=1
- added joint 44_to_33: type revolute, parent 33, child 44, origin xyz=0.5607100632388653 0.5633427228192782 0.10525246131887211 rpy=9.53345282286779 6.085246563263388 4.797191989166931, axis 0 1 0, limit lower=3.1415 upper=-3.1415 effort=1 velocity=1
- added joint 450_to_346: type revolute, parent 346, child 450, origin xyz=0.5607100632388653 0.5633427228192782 0.10525246131887211 rpy=23.833632057169474 6.085246563263388 4.797191989166931, axis 0 1 0, limit lower=3.1415 upper=-3.1415 effort=1 velocity=1
- added joint 452_to_351: type revolute, parent 351, child 452, origin xyz=0.5607100632388653 0.5633427228192782 0.10525246131887211 rpy=9.53345282286779 6.085246563263388 4.797191989166931, axis 0 1 0, limit lower=3.1415 upper=-3.1415 effort=1 velocity=1
- added joint 453_to_351: type revolute, parent 351, child 453, origin xyz=0.5607100632388653 0.5633427228192782 0.10525246131887211 rpy=14.300179234301686 6.085246563263388 4.797191989166931, axis 0 1 0, limit lower=3.1415 upper=-3.1415 effort=1 velocity=1
- added joint 454_to_351: type revolute, parent 351, child 454, origin xyz=0.5607100632388653 0.5633427228192782 0.10525246131887211 rpy=19.06690564573558 6.085246563263388 4.797191989166931, axis 0 1 0, limit lower=3.1415 upper=-3.1415 effort=1 velocity=1
- added joint 455_to_351: type revolute, parent 351, child 455, origin xyz=0.5607100632388653 0.5633427228192782 0.10525246131887211 rpy=23.833632057169474 6.085246563263388 4.797191989166931, axis 0 1 0, limit lower=3.1415 upper=-3.1415 effort=1 velocity=1
- added joint 457_to_356: type revolute, parent 356, child 457, origin xyz=0.5607100632388653 0.5633427228192782 0.10525246131887211 rpy=9.53345282286779 6.085246563263388 4.797191989166931, axis 0 1 0, limit lower=3.1415 upper=-3.1415 effort=1 velocity=1
- added joint 458_to_356: type revolute, parent 356, child 458, origin xyz=0.5607100632388653 0.5633427228192782 0.10525246131887211 rpy=14.300179234301686 6.085246563263388 4.797191989166931, axis 0 1 0, limit lower=3.1415 upper=-3.1415 effort=1 velocity=1
- added joint 459_to_356: type revolute, parent 356, child 459, origin xyz=0.5607100632388653 0.5633427228192782 0.10525246131887211 rpy=19.06690564573558 6.085246563263388 4.797191989166931, axis 0 1 0, limit lower=3.1415 upper=-3.1415 effort=1 velocity=1
- added joint 45_to_33: type revolute, parent 33, child 45, origin xyz=0.5607100632388653 0.5633427228192782 0.10525246131887211 rpy=14.300179234301686 6.085246563263388 4.797191989166931, axis 0 1 0, limit lower=3.1415 upper=-3.1415 effort=1 velocity=1
- added joint 460_to_356: type revolute, parent 356, child 460, origin xyz=0.5607100632388653 0.5633427228192782 0.10525246131887211 rpy=23.833632057169474 6.085246563263388 4.797191989166931, axis 0 1 0, limit lower=3.1415 upper=-3.1415 effort=1 velocity=1
- added joint 462_to_361: type revolute, parent 361, child 462, origin xyz=0.5607100632388653 0.5633427228192782 0.10525246131887211 rpy=9.53345282286779 6.085246563263388 4.797191989166931, axis 0 1 0, limit lower=3.1415 upper=-3.1415 effort=1 velocity=1
- added joint 463_to_361: type revolute, parent 361, child 463, origin xyz=0.5607100632388653 0.5633427228192782 0.10525246131887211 rpy=14.300179234301686 6.085246563263388 4.797191989166931, axis 0 1 0, limit lower=3.1415 upper=-3.1415 effort=1 velocity=1
- added joint 464_to_361: type revolute, parent 361, child 464, origin xyz=0.5607100632388653 0.5633427228192782 0.10525246131887211 rpy=19.06690564573558 6.085246563263388 4.797191989166931, axis 0 1 0, limit lower=3.1415 upper=-3.1415 effort=1 velocity=1
- added joint 465_to_361: type revolute, parent 361, child 465, origin xyz=0.5607100632388653 0.5633427228192782 0.10525246131887211 rpy=23.833632057169474 6.085246563263388 4.797191989166931, axis 0 1 0, limit lower=3.1415 upper=-3.1415 effort=1 velocity=1
- added joint 468_to_367: type revolute, parent 367, child 468, origin xyz=0.5607100632388653 0.5633427228192782 0.10525246131887211 rpy=9.53345282286779 6.085246563263388 4.797191989166931, axis 0 1 0, limit lower=3.1415 upper=-3.1415 effort=1 velocity=1
- added joint 469_to_367: type revolute, parent 367, child 469, origin xyz=0.5607100632388653 0.5633427228192782 0.10525246131887211 rpy=14.300179234301686 6.085246563263388 4.797191989166931, axis 0 1 0, limit lower=3.1415 upper=-3.1415 effort=1 velocity=1
- added joint 46_to_33: type revolute, parent 33, child 46, origin xyz=0.5607100632388653 0.5633427228192782 0.10525246131887211 rpy=19.06690564573558 6.085246563263388 4.797191989166931, axis 0 1 0, limit lower=3.1415 upper=-3.1415 effort=1 velocity=1
- added joint 470_to_367: type revolute, parent 367, child 470, origin xyz=0.5607100632388653 0.5633427228192782 0.10525246131887211 rpy=19.06690564573558 6.085246563263388 4.797191989166931, axis 0 1 0, limit lower=3.1415 upper=-3.1415 effort=1 velocity=1
- added joint 471_to_367: type revolute, parent 367, child 471, origin xyz=0.5607100632388653 0.5633427228192782 0.10525246131887211 rpy=23.833632057169474 6.085246563263388 4.797191989166931, axis 0 1 0, limit lower=3.1415 upper=-3.1415 effort=1 velocity=1
- added joint 473_to_372: type revolute, parent 372, child 473, origin xyz=0.5607100632388653 0.5633427228192782 0.10525246131887211 rpy=9.53345282286779 6.085246563263388 4.797191989166931, axis 0 1 0, limit lower=3.1415 upper=-3.1415 effort=1 velocity=1
- added joint 474_to_372: type revolute, parent 372, child 474, origin xyz=0.5607100632388653 0.5633427228192782 0.10525246131887211 rpy=14.300179234301686 6.085246563263388 4.797191989166931, axis 0 1 0, limit lower=3.1415 upper=-3.1415 effort=1 velocity=1
- added joint 475_to_372: type revolute, parent 372, child 475, origin xyz=0.5607100632388653 0.5633427228192782 0.10525246131887211 rpy=19.06690564573558 6.085246563263388 4.797191989166931, axis 0 1 0, limit lower=3.1415 upper=-3.1415 effort=1 velocity=1
- added joint 476_to_372: type revolute, parent 372, child 476, origin xyz=0.5607100632388653 0.5633427228192782 0.10525246131887211 rpy=23.833632057169474 6.085246563263388 4.797191989166931, axis 0 1 0, limit lower=3.1415 upper=-3.1415 effort=1 velocity=1
- added joint 478_to_377: type revolute, parent 377, child 478, origin xyz=0.5607100632388653 0.5633427228192782 0.10525246131887211 rpy=9.53345282286779 6.085246563263388 4.797191989166931, axis 0 1 0, limit lower=3.1415 upper=-3.1415 effort=1 velocity=1
- added joint 479_to_377: type revolute, parent 377, child 479, origin xyz=0.5607100632388653 0.5633427228192782 0.10525246131887211 rpy=14.300179234301686 6.085246563263388 4.797191989166931, axis 0 1 0, limit lower=3.1415 upper=-3.1415 effort=1 velocity=1
- added joint 47_to_33: type revolute, parent 33, child 47, origin xyz=0.5607100632388653 0.5633427228192782 0.10525246131887211 rpy=23.833632057169474 6.085246563263388 4.797191989166931, axis 0 1 0, limit lower=3.1415 upper=-3.1415 effort=1 velocity=1
- added joint 480_to_377: type revolute, parent 377, child 480, origin xyz=0.5607100632388653 0.5633427228192782 0.10525246131887211 rpy=19.06690564573558 6.085246563263388 4.797191989166931, axis 0 1 0, limit lower=3.1415 upper=-3.1415 effort=1 velocity=1
- added joint 481_to_377: type revolute, parent 377, child 481, origin xyz=0.5607100632388653 0.5633427228192782 0.10525246131887211 rpy=23.833632057169474 6.085246563263388 4.797191989166931, axis 0 1 0, limit lower=3.1415 upper=-3.1415 effort=1 velocity=1
- added joint 483_to_382: type revolute, parent 382, child 483, origin xyz=0.5607100632388653 0.5633427228192782 0.10525246131887211 rpy=9.53345282286779 6.085246563263388 4.797191989166931, axis 0 1 0, limit lower=3.1415 upper=-3.1415 effort=1 velocity=1
- added joint 484_to_382: type revolute, parent 382, child 484, origin xyz=0.5607100632388653 0.5633427228192782 0.10525246131887211 rpy=14.300179234301686 6.085246563263388 4.797191989166931, axis 0 1 0, limit lower=3.1415 upper=-3.1415 effort=1 velocity=1
- added joint 485_to_382: type revolute, parent 382, child 485, origin xyz=0.5607100632388653 0.5633427228192782 0.10525246131887211 rpy=19.06690564573558 6.085246563263388 4.797191989166931, axis 0 1 0, limit lower=3.1415 upper=-3.1415 effort=1 velocity=1
- added joint 486_to_382: type revolute, parent 382, child 486, origin xyz=0.5607100632388653 0.5633427228192782 0.10525246131887211 rpy=23.833632057169474 6.085246563263388 4.797191989166931, axis 0 1 0, limit lower=3.1415 upper=-3.1415 effort=1 velocity=1
- added joint 49_to_38: type revolute, parent 38, child 49, origin xyz=0.5607100632388653 0.5633427228192782 0.10525246131887211 rpy=9.53345282286779 6.085246563263388 4.797191989166931, axis 0 1 0, limit lower=3.1415 upper=-3.1415 effort=1 velocity=1
- joint 11_to_0: axis 0 1 0 -> 0 0 1; origin xyz=0.24745488733666288 0.1736730759022148 0.09603908199303623 rpy=0.47454964646738806 4.906785901388561 3.7299760154031625 -> xyz=0.15038454251742672 0.9250536779485011 0.2625608772024355 rpy=3.3579622650107432 6.158822008435018 5.754327538697678
