Commit message: added roulette wheel for choosing the parent for new generation

File: test.urdf (robot description, URDF)
Before this commit: robot pepe, 87 links, 86 joints
Links:
- removed link 144
- removed link 22
- removed link 223
- removed link 245
- removed link 266
- removed link 313
- removed link 318
- removed link 324
- removed link 329
- removed link 33
- removed link 334
- removed link 339
- removed link 346
- removed link 351
- removed link 356
- removed link 361
- removed link 367
- removed link 372
- removed link 377
- removed link 38
- removed link 382
- removed link 410
- removed link 411
- removed link 412
- removed link 414
- removed link 415
- removed link 416
- removed link 417
- removed link 419
- removed link 420
- removed link 421
- removed link 422
- removed link 425
- removed link 426
- removed link 427
- removed link 428
- removed link 430
- removed link 431
- removed link 432
- removed link 433
- removed link 435
- removed link 436
- removed link 437
- removed link 438
- removed link 44
- removed link 440
- removed link 441
- removed link 442
- removed link 443
- removed link 447
- removed link 448
- removed link 449
- removed link 45
- removed link 450
- removed link 452
- removed link 453
- removed link 454
- removed link 455
- removed link 457
- removed link 458
- removed link 459
- removed link 46
- removed link 460
- removed link 462
- removed link 463
- removed link 464
- removed link 465
- removed link 468
- removed link 469
- removed link 47
- removed link 470
- removed link 471
- removed link 473
- removed link 474
- removed link 475
- removed link 476
- removed link 478
- removed link 479
- removed link 480
- removed link 481
- removed link 483
- removed link 484
- removed link 485
- removed link 486
- removed link 49
- added link 12, mass 1.372992422681343; collision cylinder length=0.7770112710119967 radius=0.7499727342204879; visual cylinder length=0.7770112710119967 radius=0.7499727342204879
- added link 13, mass 1.372992422681343; collision cylinder length=0.7770112710119967 radius=0.7499727342204879; visual cylinder length=0.7770112710119967 radius=0.7499727342204879
- added link 14, mass 1.372992422681343; collision cylinder length=0.7770112710119967 radius=0.7499727342204879; visual cylinder length=0.7770112710119967 radius=0.7499727342204879
- link 0: mass 0.0005252686028896167 -> 1.0373343301924696; geometry collision cylinder length=0.4300649945269336 radius=0.8762285346357674; visual cylinder length=0.4300649945269336 radius=0.8762285346357674
- link 11: mass 0.033049315320639795 -> 1.372992422681343; geometry collision cylinder length=0.7770112710119967 radius=0.7499727342204879; visual cylinder length=0.7770112710119967 radius=0.7499727342204879
Joints:
- removed joint 144_to_0
- removed joint 223_to_11
- removed joint 22_to_11
- removed joint 245_to_144
- removed joint 266_to_144
- removed joint 313_to_22
- removed joint 318_to_22
- removed joint 324_to_223
- removed joint 329_to_223
- removed joint 334_to_223
- removed joint 339_to_223
- removed joint 33_to_22
- removed joint 346_to_245
- removed joint 351_to_245
- removed joint 356_to_245
- removed joint 361_to_245
- removed joint 367_to_266
- removed joint 372_to_266
- removed joint 377_to_266
- removed joint 382_to_266
- removed joint 38_to_22
- removed joint 410_to_38
- removed joint 411_to_38
- removed joint 412_to_38
- removed joint 414_to_313
- removed joint 415_to_313
- removed joint 416_to_313
- removed joint 417_to_313
- removed joint 419_to_318
- removed joint 420_to_318
- removed joint 421_to_318
- removed joint 422_to_318
- removed joint 425_to_324
- removed joint 426_to_324
- removed joint 427_to_324
- removed joint 428_to_324
- removed joint 430_to_329
- removed joint 431_to_329
- removed joint 432_to_329
- removed joint 433_to_329
- removed joint 435_to_334
- removed joint 436_to_334
- removed joint 437_to_334
- removed joint 438_to_334
- removed joint 440_to_339
- removed joint 441_to_339
- removed joint 442_to_339
- removed joint 443_to_339
- removed joint 447_to_346
- removed joint 448_to_346
- removed joint 449_to_346
- removed joint 44_to_33
- removed joint 450_to_346
- removed joint 452_to_351
- removed joint 453_to_351
- removed joint 454_to_351
- removed joint 455_to_351
- removed joint 457_to_356
- removed joint 458_to_356
- removed joint 459_to_356
- removed joint 45_to_33
- removed joint 460_to_356
- removed joint 462_to_361
- removed joint 463_to_361
- removed joint 464_to_361
- removed joint 465_to_361
- removed joint 468_to_367
- removed joint 469_to_367
- removed joint 46_to_33
- removed joint 470_to_367
- removed joint 471_to_367
- removed joint 473_to_372
- removed joint 474_to_372
- removed joint 475_to_372
- removed joint 476_to_372
- removed joint 478_to_377
- removed joint 479_to_377
- removed joint 47_to_33
- removed joint 480_to_377
- removed joint 481_to_377
- removed joint 483_to_382
- removed joint 484_to_382
- removed joint 485_to_382
- removed joint 486_to_382
- removed joint 49_to_38
- added joint 12_to_0: type revolute, parent 0, child 12, origin xyz=0.8375662920681625 0.8781208897108024 0.20189983192874617 rpy=1.644234303537614 0.819126464931671 3.201727369301795, axis 0 1 0, limit lower=3.1415 upper=-3.1415 effort=1 velocity=1
- added joint 13_to_0: type revolute, parent 0, child 13, origin xyz=0.8375662920681625 0.8781208897108024 0.20189983192874617 rpy=2.1923124047168185 0.819126464931671 3.201727369301795, axis 0 1 0, limit lower=3.1415 upper=-3.1415 effort=1 velocity=1
- added joint 14_to_0: type revolute, parent 0, child 14, origin xyz=0.8375662920681625 0.8781208897108024 0.20189983192874617 rpy=2.7403905058960234 0.819126464931671 3.201727369301795, axis 0 1 0, limit lower=3.1415 upper=-3.1415 effort=1 velocity=1
- joint 11_to_0: axis 0 0 1 -> 0 1 0; origin xyz=0.15038454251742672 0.9250536779485011 0.2625608772024355 rpy=3.3579622650107432 6.158822008435018 5.754327538697678 -> xyz=0.8375662920681625 0.8781208897108024 0.20189983192874617 rpy=1.0961562023584093 0.819126464931671 3.201727369301795
